File: KiCad Project/Omni_X_LT_board.kicad_sch (KiCad schematic)
At the start: 32 parts, among them J1 Conn_01x02_Female, J2 Conn_01x02_Female, U1 TLV9001IDCK, U2 TLV9001IDCK, U3 ADS1110

Commit message: update KiCad files
Parts:
- R2: value 1k -> 7.5k; MPN ESR10EZPF1001 -> ESR10EZPF7501
Connections:
- net +3V3: now reaches XA1.3V3 (3.3V)
- net +3V3: now also C10.1, R1.1, R14.1, R15.1, U1.5 (V+), U2.5 (V+), U3.5 (VDD)
- removed net +5V: C10.1, R1.1, R14.1, R15.1, U1.5 (V+), U2.5 (V+), U3.5 (VDD), XA1.5V
