File: hardware/KiCad Project/GS-One_IoT_board/GS-One_IoT_board.kicad_pcb (KiCad board)
At the start: 2 copper layers, 50.9 x 22.9 mm, 33 parts, among them J1 Conn_01x02_Female, J2 Conn_01x02_Female, U1 TLV9001IDCK, U2 TLV9001IDCK

Commit message: final version v0.1 for hardware
Parts:
- C9: value 100u -> 2.2u; footprint Capacitor_SMD:C_1206_3216Metric -> Capacitor_SMD:C_0603_1608Metric
Routing:
- net Net-(C9-Pad1): track 8.18 -> 8.88 mm
Other:
- board text added: "CITI Lab SASTRESS Project Regis Rousseau 2024 v0.1"
- board text added: "GS-ONE"
- board text removed: "CITI Lab SASTRESS Prj Regis Rousseau"
- board text removed: "GS-One"
Changed lines of the file:
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@@
     (descr "JST PH series connector, B2B-PH-SM4-TB (http://www.jst-mfg.com/product/pdf/eng/ePH.pdf), generated with kicad-footprint-generator")
     (tags "connector JST PH side entry")
+    (property "MPN" "B2B-PH-SM4-TB(LF)(SN)")
+    (property "Manufacturer" "JST Sales America Inc")
     (property "Sheetfile" "GS-One_IoT_board.kicad_sch")
     (property "Sheetname" "")
@@
     )
   )
-  (footprint "Capacitor_SMD:C_1206_3216Metric" (layer "F.Cu")
+  (footprint "Capacitor_SMD:C_0603_1608Metric" (layer "F.Cu")
     (at 104.648 54.737 -90)
-    (descr "Capacitor SMD 1206 (3216 Metric), square (rectangular) end terminal, IPC_7351 nominal, (Body size source: IPC-SM-782 page 76, https://www.pcb-3d.com/wordpress/wp-content/uploads/ipc-sm-782a_amendment_1_and_2.pdf), generated with kicad-footprint-generator")
+    (descr "Capacitor SMD 0603 (1608 Metric), square (rectangular) end terminal, IPC_7351 nominal, (Body size source: IPC-SM-782 page 76, https://www.pcb-3d.com/wordpress/wp-content/uploads/ipc-sm-782a_amendment_1_and_2.pdf), generated with kicad-footprint-generator")
     (tags "capacitor")
-    (property "MPN" "GRM31CD80J107MEA8K")
+    (property "MPN" "GRM188R61E106KA73J")
     (property "Manufacturer" "Murata Electronics")
     (property "Sheetfile" "GS-One_IoT_board.kicad_sch")
     (property "Sheetname" "")
     (attr smd)
-    (fp_text reference "C9" (at 1.524 -1.778 90) (layer "F.SilkS") hide
-      (effects (font (size 1 1) (thickness 0.15)))
-    )
-    (fp_text value "100u" (at 0 1.85 90) (layer "F.Fab") hide
-      (effects (font (size 1 1) (thickness 0.15)))
-    )
-    (fp_text user "${REFERENCE}" (at 0 0 90) (layer "F.Fab")
-      (effects (font (size 0.8 0.8) (thickness 0.12)))
-    )
-    (fp_line (start -0.711252 -0.91) (end 0.711252 -0.91) (layer "F.SilkS") (width 0.12))
-    (fp_line (start -0.711252 0.91) (end 0.711252 0.91) (layer "F.SilkS") (width 0.12))
-    (fp_line (start -2.3 1.15) (end -2.3 -1.15) (layer "F.CrtYd") (width 0.05))
-    (fp_line (start 2.3 1.15) (end -2.3 1.15) (layer "F.CrtYd") (width 0.05))
-    (fp_line (start 2.3 -1.15) (end 2.3 1.15) (layer "F.CrtYd") (width 0.05))
-    (fp_line (start -2.3 -1.15) (end 2.3 -1.15) (layer "F.CrtYd") (width 0.05))
-    (fp_line (start 1.6 -0.8) (end 1.6 0.8) (layer "F.Fab") (width 0.1))
-    (fp_line (start -1.6 0.8) (end -1.6 -0.8) (layer "F.Fab") (width 0.1))
-    (fp_line (start 1.6 0.8) (end -1.6 0.8) (layer "F.Fab") (width 0.1))
-    (fp_line (start -1.6 -0.8) (end 1.6 -0.8) (layer "F.Fab") (width 0.1))
-    (pad "1" smd roundrect locked (at -1.475 0 270) (size 1.15 1.8) (layers "F.Cu" "F.Paste" "F.Mask") (roundrect_rratio 0.217391)
+    (fp_text reference "C9" (at 0 -1.43 -90) (layer "F.SilkS") hide
+      (effects (font (size 1 1) (thickness 0.15)))
+    )
+    (fp_text value "2.2u" (at 0 1.43 -90) (layer "F.Fab") hide
+      (effects (font (size 1 1) (thickness 0.15)))
+    )
+    (fp_text user "${REFERENCE}" (at 0 0 -90) (layer "F.Fab")
+      (effects (font (size 0.4 0.4) (thickness 0.06)))
+    )
+    (fp_line (start -0.14058 -0.51) (end 0.14058 -0.51) (layer "F.SilkS") (width 0.12))
+    (fp_line (start -0.14058 0.51) (end 0.14058 0.51) (layer "F.SilkS") (width 0.12))
+    (fp_line (start 1.48 -0.73) (end 1.48 0.73) (layer "F.CrtYd") (width 0.05))
+    (fp_line (start 1.48 0.73) (end -1.48 0.73) (layer "F.CrtYd") (width 0.05))
+    (fp_line (start -1.48 -0.73) (end 1.48 -0.73) (layer "F.CrtYd") (width 0.05))
+    (fp_line (start -1.48 0.73) (end -1.48 -0.73) (layer "F.CrtYd") (width 0.05))
+    (fp_line (start 0.8 0.4) (end -0.8 0.4) (layer "F.Fab") (width 0.1))
+    (fp_line (start -0.8 0.4) (end -0.8 -0.4) (layer "F.Fab") (width 0.1))
+    (fp_line (start -0.8 -0.4) (end 0.8 -0.4) (layer "F.Fab") (width 0.1))
+    (fp_line (start 0.8 -0.4) (end 0.8 0.4) (layer "F.Fab") (width 0.1))
+    (pad "1" smd roundrect locked (at -0.775 0 270) (size 0.9 0.95) (layers "F.Cu" "F.Paste" "F.Mask") (roundrect_rratio 0.25)
       (net 13 "Net-(C9-Pad1)") (pintype "passive"))
-    (pad "2" smd roundrect locked (at 1.475 0 270) (size 1.15 1.8) (layers "F.Cu" "F.Paste" "F.Mask") (roundrect_rratio 0.217391)
+    (pad "2" smd roundrect locked (at 0.775 0 270) (size 0.9 0.95) (layers "F.Cu" "F.Paste" "F.Mask") (roundrect_rratio 0.25)
       (net 2 "GND") (pintype "passive"))
-    (model "${KICAD6_3DMODEL_DIR}/Capacitor_SMD.3dshapes/C_1206_3216Metric.wrl"
+    (model "${KICAD6_3DMODEL_DIR}/Capacitor_SMD.3dshapes/C_0603_1608Metric.wrl"
       (offset (xyz 0 0 0))
       (scale (xyz 1 1 1))
@@
   )
   (gr_rect (start 97.155 41.275) (end 148.082 64.135) (layer "Edge.Cuts") (width 0.1) (fill none))
-  (gr_text "GS-One" (at 141.224 55.372) (layer "F.SilkS")
-    (effects (font (size 1 1) (thickness 0.15)))
+  (gr_text "GS-ONE" (at 142.494 55.626) (layer "F.SilkS")
+    (effects (font (size 0.5 0.5) (thickness 0.125)))
   )
   (gr_text "ADC0" (at 121.412 61.468) (layer "F.SilkS")
@@
     (effects (font (size 0.5 0.5) (thickness 0.125)))
   )
-  (gr_text "CITI Lab\nSASTRESS Prj\nRegis Rousseau" (at 137.795 48.006) (layer "F.SilkS")
-    (effects (font (size 0.8 0.8) (thickness 0.15)) (justify left))
+  (gr_text "CITI Lab\nSASTRESS Project\nRegis Rousseau\n2024 v0.1" (at 137.668 49.276) (layer "F.SilkS")
+    (effects (font (size 0.6 0.6) (thickness 0.125)) (justify left))
   )
   (gr_text "234Hz LP" (at 130.302 57.658) (layer "F.SilkS")
@@
   (segment (start 104.648 53.262) (end 107.999 53.262) (width 0.2) (layer "F.Cu") (net 13))
   (segment (start 107.999 53.262) (end 108.077 53.34) (width 0.2) (layer "F.Cu") (net 13))
+  (segment (start 104.648 53.262) (end 104.648 53.962) (width 0.2) (layer "F.Cu") (net 13))
   (segment (start 102.3947 53.262) (end 104.648 53.262) (width 0.2) (layer "F.Cu") (net 13))
   (segment (start 128.458 47.076) (end 127.7803 47.076) (width 0.4) (layer "F.Cu") (net 14))
