File: hardware/KiCad Project/GS-One_IoT_board/GS-One_IoT_board.kicad_sch (KiCad schematic)
At the start: 33 parts, among them J1 Conn_01x02_Female, J2 Conn_01x02_Female, U1 TLV9001IDCK, U2 TLV9001IDCK

Commit message: final version v0.1 for hardware
Parts:
- C9: value 100u -> 2.2u; footprint Capacitor_SMD:C_1206_3216Metric -> Capacitor_SMD:C_0603_1608Metric; MPN GRM31CD80J107MEA8K -> GRM188R61E106KA73J
Changed lines of the file:
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@@
       (effects (font (size 1.27 1.27)) (justify left))
     )
-    (property "Value" "100u" (id 1) (at 244.856 111.8869 0)
-      (effects (font (size 1.27 1.27)) (justify left))
-    )
-    (property "Footprint" "Capacitor_SMD:C_1206_3216Metric" (id 2) (at 242.0112 115.316 0)
+    (property "Value" "2.2u" (id 1) (at 244.856 111.8869 0)
+      (effects (font (size 1.27 1.27)) (justify left))
+    )
+    (property "Footprint" "Capacitor_SMD:C_0603_1608Metric" (id 2) (at 242.0112 115.316 0)
       (effects (font (size 1.27 1.27)) hide)
     )
@@
       (effects (font (size 1.27 1.27)) hide)
     )
-    (property "MPN" "GRM31CD80J107MEA8K" (id 5) (at 241.046 111.506 0)
+    (property "MPN" "GRM188R61E106KA73J" (id 5) (at 241.046 111.506 0)
       (effects (font (size 1.27 1.27)) hide)
     )
@@
     )
     (path "/449c07cf-fab5-4a92-b79f-389a24082a2c"
-      (reference "C9") (unit 1) (value "100u") (footprint "Capacitor_SMD:C_1206_3216Metric")
+      (reference "C9") (unit 1) (value "2.2u") (footprint "Capacitor_SMD:C_0603_1608Metric")
     )
     (path "/f33fd41a-ecc2-4ad8-8e78-e42925e5e442"
